File: Circuits_Schema/Kicad/Satellite_Circuit/Satellite_Circuit.kicad_sch (KiCad schematic)
At the start: 11 parts, among them U1 BNO055, Y1 32.768kHZ

Commit message: MCU model added and first connexions were made
Parts:
- added IC1: MBED-LPC1768, DIPS2286W63P254L5370H300Q40N, symbol MBED-LPC1768:MBED-LPC1768
Connections:
- net Earth: now also IC1.1 (GND)
- net SCL: now also IC1.10 (DIP10)
- net SDA: now also IC1.9 (DIP9)
- net VDDIO: now reaches C2.2, C3.2, R1.1, R2.1, R3.2, U1.11 (~{RESET}), U1.28 (VDDIO)
- net VDDIO: now also IC1.40 (EXT_3V3)
Changed lines of the file:
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@@
   (junction (at 71.12 31.75) (diameter 0) (color 0 0 0 0)
   )
+  (junction (at 54.61 63.5) (diameter 0) (color 0 0 0 0)
+  )
   (junction (at 54.61 67.31) (diameter 0) (color 0 0 0 0)
   )
@@
   (junction (at 62.23 67.31) (diameter 0) (color 0 0 0 0)
   )
+  (wire (pts (xy 54.61 63.5) (xy 54.61 67.31))
+    (stroke (width 0) (type default))
+  )
+  (wire (pts (xy 105.41 26.67) (xy 110.49 26.67))
+    (stroke (width 0) (type default))
+  )
   (wire (pts (xy 41.91 73.66) (xy 41.91 64.77))
     (stroke (width 0) (type default))
@@
     (stroke (width 0) (type default))
   )
-  (wire (pts (xy 54.61 62.23) (xy 54.61 67.31))
+  (wire (pts (xy 54.61 62.23) (xy 54.61 63.5))
     (stroke (width 0) (type default))
   )
@@
     (stroke (width 0) (type default))
   )
+  (wire (pts (xy 54.61 63.5) (xy 58.42 63.5))
+    (stroke (width 0) (type default))
+  )
   (wire (pts (xy 36.83 57.15) (xy 34.29 57.15))
     (stroke (width 0) (type default))
   )
+  (wire (pts (xy 153.67 26.67) (xy 160.02 26.67))
+    (stroke (width 0) (type default))
+  )
   (wire (pts (xy 49.53 67.31) (xy 54.61 67.31))
     (stroke (width 0) (type default))
@@
     (stroke (width 0) (type default))
   )
+  (wire (pts (xy 99.06 49.53) (xy 110.49 49.53))
+    (stroke (width 0) (type default))
+  )
   (wire (pts (xy 54.61 77.47) (xy 58.42 77.47))
     (stroke (width 0) (type default))
@@
     (stroke (width 0) (type default))
   )
+  (wire (pts (xy 102.87 46.99) (xy 110.49 46.99))
+    (stroke (width 0) (type default))
+  )
   (wire (pts (xy 71.12 44.45) (xy 71.12 41.91))
     (stroke (width 0) (type default))
@@
   (wire (pts (xy 30.48 54.61) (xy 30.48 67.31))
     (stroke (width 0) (type default))
+  )
+  (label "SCL" (at 101.6 49.53 180) (fields_autoplaced)
+    (effects (font (size 1.27 1.27)) (justify right bottom))
+  )
+  (label "GND" (at 106.68 26.67 0) (fields_autoplaced)
+    (effects (font (size 1.27 1.27)) (justify left bottom))
+  )
+  (label "GND" (at 57.15 63.5 0) (fields_autoplaced)
+    (effects (font (size 1.27 1.27)) (justify left bottom))
   )
   (label "I2C_ADDR" (at 34.29 72.39 270) (fields_autoplaced)
     (effects (font (size 1.27 1.27)) (justify right bottom))
   )
+  (label "VDDIO" (at 156.21 26.67 0) (fields_autoplaced)
+    (effects (font (size 1.27 1.27)) (justify left bottom))
+  )
   (label "INT" (at 34.29 26.67 270) (fields_autoplaced)
     (effects (font (size 1.27 1.27)) (justify right bottom))
@@
     (effects (font (size 1.27 1.27)) (justify right bottom))
   )
+  (label "SDA" (at 105.41 46.99 180) (fields_autoplaced)
+    (effects (font (size 1.27 1.27)) (justify right bottom))
+  )
   (label "SDA" (at 24.13 53.34 90) (fields_autoplaced)
+    (effects (font (size 1.27 1.27)) (justify left bottom))
+  )
+  (label "VDDIO" (at 57.15 22.86 0) (fields_autoplaced)
     (effects (font (size 1.27 1.27)) (justify left bottom))
   )
@@
         )
       )
+    )
+  )
+  (symbol (lib_id "MBED-LPC1768:MBED-LPC1768") (at 110.49 26.67 0) (unit 1)
+    (in_bom yes) (on_board yes) (dnp no) (fields_autoplaced)
+    (property "Reference" "IC1" (at 132.08 20.32 0)
+      (effects (font (size 1.27 1.27)))
+    )
+    (property "Value" "MBED-LPC1768" (at 132.08 22.86 0)
+      (effects (font (size 1.27 1.27)))
+    )
+    (property "Footprint" "DIPS2286W63P254L5370H300Q40N" (at 149.86 121.59 0)
+      (effects (font (size 1.27 1.27)) (justify left top) hide)
+    )
+    (property "Datasheet" "https://os.mbed.com/platforms/mbed-LPC1768/" (at 149.86 221.59 0)
+      (effects (font (size 1.27 1.27)) (justify left top) hide)
+    )
+    (property "Height" "3" (at 149.86 421.59 0)
+      (effects (font (size 1.27 1.27)) (justify left top) hide)
+    )
+    (property "Manufacturer_Name" "mbed" (at 149.86 521.59 0)
+      (effects (font (size 1.27 1.27)) (justify left top) hide)
+    )
+    (property "Manufacturer_Part_Number" "MBED-LPC1768" (at 149.86 621.59 0)
+      (effects (font (size 1.27 1.27)) (justify left top) hide)
+    )
+    (property "Mouser Part Number" "" (at 149.86 721.59 0)
+      (effects (font (size 1.27 1.27)) (justify left top) hide)
+    )
+    (property "Mouser Price/Stock" "" (at 149.86 821.59 0)
+      (effects (font (size 1.27 1.27)) (justify left top) hide)
+    )
+    (property "Arrow Part Number" "" (at 149.86 921.59 0)
+      (effects (font (size 1.27 1.27)) (justify left top) hide)
+    )
+    (property "Arrow Price/Stock" "" (at 149.86 1021.59 0)
+      (effects (font (size 1.27 1.27)) (justify left top) hide)
+    )
+    (pin "1")
+    (pin "10")
+    (pin "11")
+    (pin "12")
+    (pin "13")
+    (pin "14")
+    (pin "15")
+    (pin "16")
+    (pin "17")
+    (pin "18")
+    (pin "19")
+    (pin "2")
+    (pin "20")
+    (pin "21")
+    (pin "22")
+    (pin "23")
+    (pin "24")
+    (pin "25")
+    (pin "26")
+    (pin "27")
+    (pin "28")
+    (pin "29")
+    (pin "3")
+    (pin "30")
+    (pin "31")
+    (pin "32")
+    (pin "33")
+    (pin "34")
+    (pin "35")
+    (pin "36")
+    (pin "37")
+    (pin "38")
+    (pin "39")
+    (pin "4")
+    (pin "40")
+    (pin "5")
+    (pin "6")
+    (pin "7")
+    (pin "8")
+    (pin "9")
+    (instances
+      (project "Satellite_Circuit"
+        (path "/1ba48872-20f1-4135-8850-dcaa1bdd8874"
+          (reference "IC1") (unit 1)
+        )
+      )

Commit message: Cam model added(no connections still), temperature sensor added and connected (p8)
Parts:
- added R4: 4.7k, symbol Device:R
- added U2: ESP32-CAM, ESP32-CAM, symbol ESP32-CAM:ESP32-CAM
- added U3: DS18B20, Package_TO_SOT_THT:TO-92_Inline, symbol Sensor_Temperature:DS18B20
Connections:
- net Earth: now also U2.12 (GND_2), U3.1 (GND)
- net VDDIO: now also R4.1, U2.9 (3V3), U3.3 (V_{DD})
- net Temp_int: now reaches IC1.8 (DIP8)
- net Temp_int: now also R4.2, U3.2 (DQ)
Changed lines of the file:
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@@
 (kicad_sch (version 20230121) (generator eeschema)
   (paper "A4")
+  (junction (at 85.09 101.6) (diameter 0) (color 0 0 0 0)
+  )
   (junction (at 73.66 54.61) (diameter 0) (color 0 0 0 0)
   )
@@
   (junction (at 49.53 64.77) (diameter 0) (color 0 0 0 0)
   )
+  (junction (at 76.2 91.44) (diameter 0) (color 0 0 0 0)
+  )
   (junction (at 88.9 38.1) (diameter 0) (color 0 0 0 0)
   )
@@
     (stroke (width 0) (type default))
   )
+  (wire (pts (xy 76.2 91.44) (xy 76.2 93.98))
+    (stroke (width 0) (type default))
+  )
   (wire (pts (xy 83.82 82.55) (xy 58.42 82.55))
     (stroke (width 0) (type default))
@@
     (stroke (width 0) (type default))
   )
+  (wire (pts (xy 85.09 101.6) (xy 88.9 101.6))
+    (stroke (width 0) (type default))
+  )
   (wire (pts (xy 88.9 38.1) (xy 90.17 38.1))
     (stroke (width 0) (type default))
@@
     (stroke (width 0) (type default))
   )
+  (wire (pts (xy 83.82 101.6) (xy 85.09 101.6))
+    (stroke (width 0) (type default))
+  )
   (wire (pts (xy 36.83 22.86) (xy 36.83 31.75))
     (stroke (width 0) (type default))
@@
     (stroke (width 0) (type default))
   )
+  (wire (pts (xy 85.09 99.06) (xy 85.09 101.6))
+    (stroke (width 0) (type default))
+  )
   (wire (pts (xy 67.31 44.45) (xy 71.12 44.45))
     (stroke (width 0) (type default))
@@
     (stroke (width 0) (type default))
   )
+  (wire (pts (xy 76.2 91.44) (xy 85.09 91.44))
+    (stroke (width 0) (type default))
+  )
   (wire (pts (xy 54.61 22.86) (xy 83.82 22.86))
     (stroke (width 0) (type default))
@@
     (stroke (width 0) (type default))
   )
+  (wire (pts (xy 76.2 88.9) (xy 76.2 91.44))
+    (stroke (width 0) (type default))
+  )
   (wire (pts (xy 36.83 57.15) (xy 34.29 57.15))
     (stroke (width 0) (type default))
@@
     (stroke (width 0) (type default))
   )
+  (wire (pts (xy 50.8 105.41) (xy 53.34 105.41))
+    (stroke (width 0) (type default))
+  )
   (wire (pts (xy 99.06 49.53) (xy 110.49 49.53))
     (stroke (width 0) (type default))
@@
     (stroke (width 0) (type default))
   )
+  (wire (pts (xy 110.49 44.45) (xy 97.79 44.45))
+    (stroke (width 0) (type default))
+  )
   (wire (pts (xy 17.78 19.05) (xy 45.72 19.05))
     (stroke (width 0) (type default))
   )
+  (wire (pts (xy 50.8 97.79) (xy 55.88 97.79))
+    (stroke (width 0) (type default))
+  )
   (wire (pts (xy 34.29 57.15) (xy 34.29 74.93))
     (stroke (width 0) (type default))
@@
     (stroke (width 0) (type default))
   )
+  (wire (pts (xy 97.79 43.18) (xy 97.79 44.45))
+    (stroke (width 0) (type default))
+  )
   (wire (pts (xy 49.53 21.59) (xy 49.53 26.67))
     (stroke (width 0) (type default))
@@
   (wire (pts (xy 30.48 54.61) (xy 30.48 67.31))
     (stroke (width 0) (type default))
+  )
+  (label "Temp_int" (at 88.9 101.6 0) (fields_autoplaced)
+    (effects (font (size 1.27 1.27)) (justify left bottom))
+  )
+  (label "GND" (at 53.34 105.41 0) (fields_autoplaced)
+    (effects (font (size 1.27 1.27)) (justify left bottom))
   )
   (label "SCL" (at 101.6 49.53 180) (fields_autoplaced)
@@
     (effects (font (size 1.27 1.27)) (justify left bottom))
   )
+  (label "GND" (at 76.2 109.22 0) (fields_autoplaced)
+    (effects (font (size 1.27 1.27)) (justify left bottom))
+  )
   (label "GND" (at 57.15 63.5 0) (fields_autoplaced)
     (effects (font (size 1.27 1.27)) (justify left bottom))
@@
     (effects (font (size 1.27 1.27)) (justify right bottom))
   )
+  (label "VDDIO" (at 55.88 97.79 0) (fields_autoplaced)
+    (effects (font (size 1.27 1.27)) (justify left bottom))
+  )
   (label "VDDIO" (at 156.21 26.67 0) (fields_autoplaced)
     (effects (font (size 1.27 1.27)) (justify left bottom))
@@
   )
   (label "VDDIO" (at 57.15 22.86 0) (fields_autoplaced)
+    (effects (font (size 1.27 1.27)) (justify left bottom))
+  )
+  (label "Temp_int" (at 97.79 43.18 0) (fields_autoplaced)
+    (effects (font (size 1.27 1.27)) (justify left bottom))
+  )
+  (label "VDDIO" (at 76.2 88.9 0) (fields_autoplaced)
     (effects (font (size 1.27 1.27)) (justify left bottom))
   )
@@
         (path "/1ba48872-20f1-4135-8850-dcaa1bdd8874"
           (reference "U1") (unit 1)
+        )
+      )
+    )
+  )
+  (symbol (lib_id "Device:R") (at 85.09 95.25 0) (unit 1)
+    (in_bom yes) (on_board yes) (dnp no) (fields_autoplaced)
+    (property "Reference" "R4" (at 87.63 94.615 0)
+      (effects (font (size 1.27 1.27)) (justify left))
+    )
+    (property "Value" "4.7k" (at 87.63 97.155 0)
+      (effects (font (size 1.27 1.27)) (justify left))
+    )
+    (property "Footprint" "" (at 83.312 95.25 90)
+      (effects (font (size 1.27 1.27)) hide)
+    )
+    (property "Datasheet" "~" (at 85.09 95.25 0)
+      (effects (font (size 1.27 1.27)) hide)
+    )
+    (pin "1")
+    (pin "2")
+    (instances
+      (project "Satellite_Circuit"
+        (path "/1ba48872-20f1-4135-8850-dcaa1bdd8874"
+          (reference "R4") (unit 1)
         )
       )
@@
     )
   )
+  (symbol (lib_id "Sensor_Temperature:DS18B20") (at 76.2 101.6 0) (unit 1)
+    (in_bom yes) (on_board yes) (dnp no) (fields_autoplaced)
+    (property "Reference" "U3" (at 69.85 100.965 0)
+      (effects (font (size 1.27 1.27)) (justify right))
+    )
+    (property "Value" "DS18B20" (at 69.85 103.505 0)
+      (effects (font (size 1.27 1.27)) (justify right))
+    )
+    (property "Footprint" "Package_TO_SOT_THT:TO-92_Inline" (at 50.8 107.95 0)
+      (effects (font (size 1.27 1.27)) hide)
+    )
+    (property "Datasheet" "http://datasheets.maximintegrated.com/en/ds/DS18B20.pdf" (at 72.39 95.25 0)
+      (effects (font (size 1.27 1.27)) hide)
+    )
+    (pin "1")
+    (pin "2")
+    (pin "3")
+    (instances
+      (project "Satellite_Circuit"
+        (path "/1ba48872-20f1-4135-8850-dcaa1bdd8874"
+          (reference "U3") (unit 1)
+        )
+      )
+    )
+  )
   (symbol (lib_id "Device:R") (at 29.21 38.1 0) (unit 1)
     (in_bom yes) (on_board yes) (dnp no) (fields_autoplaced)
@@
         )
       )
+    )
+  )
+  (symbol (lib_id "ESP32-CAM:ESP32-CAM") (at 20.32 97.79 0) (unit 1)
+    (in_bom yes) (on_board yes) (dnp no) (fields_autoplaced)
+    (property "Reference" "U2" (at 35.56 91.44 0)
+      (effects (font (size 1.27 1.27)))
+    )
+    (property "Value" "ESP32-CAM" (at 35.56 93.98 0)
+      (effects (font (size 1.27 1.27)))
+    )
+    (property "Footprint" "ESP32-CAM" (at 20.32 97.79 0)
+      (effects (font (size 1.27 1.27)) (justify bottom) hide)
+    )
+    (property "Datasheet" "" (at 20.32 97.79 0)
+      (effects (font (size 1.27 1.27)) hide)
+    )
+    (property "ARROW_PART_NUMBER" "" (at 20.32 97.79 0)
+      (effects (font (size 1.27 1.27)) (justify bottom) hide)
+    )
+    (property "MOUSER_PART_NUMBER" "" (at 20.32 97.79 0)
+      (effects (font (size 1.27 1.27)) (justify bottom) hide)
+    )
+    (property "ARROW_PRICE-STOCK" "" (at 20.32 97.79 0)
+      (effects (font (size 1.27 1.27)) (justify bottom) hide)
+    )
+    (property "HEIGHT" "5mm" (at 20.32 97.79 0)
+      (effects (font (size 1.27 1.27)) (justify bottom) hide)
+    )
+    (property "MANUFACTURER_NAME" "Ai-Thinker" (at 20.32 97.79 0)
+      (effects (font (size 1.27 1.27)) (justify bottom) hide)
+    )
+    (property "MANUFACTURER_PART_NUMBER" "ESP32-CAM" (at 20.32 97.79 0)
+      (effects (font (size 1.27 1.27)) (justify bottom) hide)
+    )
+    (property "MOUSER_PRICE-STOCK" "" (at 20.32 97.79 0)
+      (effects (font (size 1.27 1.27)) (justify bottom) hide)
+    )
+    (property "DESCRIPTION" "Modules PCBA Module RoHS" (at 20.32 97.79 0)
+      (effects (font (size 1.27 1.27)) (justify bottom) hide)
+    )
+    (pin "1")
+    (pin "10")
+    (pin "11")
+    (pin "12")
+    (pin "13")
+    (pin "14")
+    (pin "15")
+    (pin "16")
+    (pin "2")
+    (pin "3")
+    (pin "4")
+    (pin "5")
+    (pin "6")
+    (pin "7")
+    (pin "8")
+    (pin "9")
+    (instances
+      (project "Satellite_Circuit"
+        (path "/1ba48872-20f1-4135-8850-dcaa1bdd8874"
+          (reference "U2") (unit 1)
+        )
+      )

Commit message: Light Sensor Connected added
Parts:
- added J1: Conn_01x07, symbol Connector_Generic:Conn_01x07
Connections:
- net Earth: now also J1.7 (Pin_7)
- net VDDIO: now also J1.1 (Pin_1)
- net LS1: now reaches IC1.15 (DIP15)
- net LS1: now also J1.2 (Pin_2)
- net LS2: now reaches IC1.16 (DIP16)
- net LS2: now also J1.3 (Pin_3)
- net LS3: now reaches IC1.17 (DIP17)
- net LS3: now also J1.4 (Pin_4)
- net LS4: now reaches IC1.18 (DIP18)
- net LS4: now also J1.5 (Pin_5)
- net LS5: now reaches IC1.19 (DIP19)
- net LS5: now also J1.6 (Pin_6)
Changed lines of the file:
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@@
+    (stroke (width 0) (type default))
+  )
+  (wire (pts (xy 109.22 91.44) (xy 109.22 92.71))
     (stroke (width 0) (type default))
   )
@@
     (stroke (width 0) (type default))
   )
+  (wire (pts (xy 109.22 92.71) (xy 114.3 92.71))
+    (stroke (width 0) (type default))
+  )
   (wire (pts (xy 24.13 49.53) (xy 36.83 49.53))
     (stroke (width 0) (type default))
@@
     (stroke (width 0) (type default))
   )
+  (wire (pts (xy 105.41 64.77) (xy 110.49 64.77))
+    (stroke (width 0) (type default))
+  )
   (wire (pts (xy 76.2 91.44) (xy 76.2 93.98))
     (stroke (width 0) (type default))
@@
     (stroke (width 0) (type default))
   )
+  (wire (pts (xy 106.68 62.23) (xy 110.49 62.23))
+    (stroke (width 0) (type default))
+  )
   (wire (pts (xy 67.31 54.61) (xy 73.66 54.61))
     (stroke (width 0) (type default))
@@
     (stroke (width 0) (type default))
   )
+  (wire (pts (xy 107.95 100.33) (xy 114.3 100.33))
+    (stroke (width 0) (type default))
+  )
   (wire (pts (xy 36.83 22.86) (xy 36.83 31.75))
     (stroke (width 0) (type default))
@@
     (stroke (width 0) (type default))
   )
+  (wire (pts (xy 107.95 95.25) (xy 114.3 95.25))
+    (stroke (width 0) (type default))
+  )
+  (wire (pts (xy 105.41 69.85) (xy 110.49 69.85))
+    (stroke (width 0) (type default))
+  )
   (wire (pts (xy 76.2 91.44) (xy 85.09 91.44))
     (stroke (width 0) (type default))
@@
     (stroke (width 0) (type default))
   )
+  (wire (pts (xy 104.14 91.44) (xy 109.22 91.44))
+    (stroke (width 0) (type default))
+  )
   (wire (pts (xy 73.66 52.07) (xy 73.66 54.61))
     (stroke (width 0) (type default))
@@
     (stroke (width 0) (type default))
   )
+  (wire (pts (xy 107.95 97.79) (xy 114.3 97.79))
+    (stroke (width 0) (type default))
+  )
   (wire (pts (xy 26.67 82.55) (xy 58.42 82.55))
     (stroke (width 0) (type default))
@@
     (stroke (width 0) (type default))
   )
+  (wire (pts (xy 106.68 72.39) (xy 110.49 72.39))
+    (stroke (width 0) (type default))
+  )
   (wire (pts (xy 29.21 34.29) (xy 29.21 22.86))
     (stroke (width 0) (type default))
@@
     (stroke (width 0) (type default))
   )
+  (wire (pts (xy 107.95 109.22) (xy 107.95 107.95))
+    (stroke (width 0) (type default))
+  )
   (wire (pts (xy 17.78 19.05) (xy 45.72 19.05))
     (stroke (width 0) (type default))
@@
     (stroke (width 0) (type default))
   )
+  (wire (pts (xy 107.95 107.95) (xy 114.3 107.95))
+    (stroke (width 0) (type default))
+  )
+  (wire (pts (xy 106.68 67.31) (xy 110.49 67.31))
+    (stroke (width 0) (type default))
+  )
   (wire (pts (xy 41.91 64.77) (xy 49.53 64.77))
     (stroke (width 0) (type default))
@@
     (stroke (width 0) (type default))
   )
+  (wire (pts (xy 105.41 109.22) (xy 107.95 109.22))
+    (stroke (width 0) (type default))
+  )
   (wire (pts (xy 81.28 44.45) (xy 88.9 44.45))
     (stroke (width 0) (type default))
   )
+  (wire (pts (xy 107.95 105.41) (xy 114.3 105.41))
+    (stroke (width 0) (type default))
+  )
   (wire (pts (xy 97.79 43.18) (xy 97.79 44.45))
     (stroke (width 0) (type default))
@@
     (stroke (width 0) (type default))
   )
+  (wire (pts (xy 107.95 102.87) (xy 114.3 102.87))
+    (stroke (width 0) (type default))
+  )
   (label "Temp_int" (at 88.9 101.6 0) (fields_autoplaced)
     (effects (font (size 1.27 1.27)) (justify left bottom))
   )
+  (label "LS4" (at 107.95 102.87 180) (fields_autoplaced)
+    (effects (font (size 1.27 1.27)) (justify right bottom))
+  )
+  (label "LS2" (at 107.95 97.79 180) (fields_autoplaced)
+    (effects (font (size 1.27 1.27)) (justify right bottom))
+  )
   (label "GND" (at 53.34 105.41 0) (fields_autoplaced)
     (effects (font (size 1.27 1.27)) (justify left bottom))
@@
     (effects (font (size 1.27 1.27)) (justify right bottom))
   )
+  (label "LS1" (at 106.68 62.23 0) (fields_autoplaced)
+    (effects (font (size 1.27 1.27)) (justify left bottom))
+  )
   (label "GND" (at 106.68 26.67 0) (fields_autoplaced)
     (effects (font (size 1.27 1.27)) (justify left bottom))
   )
+  (label "LS5" (at 107.95 105.41 180) (fields_autoplaced)
+    (effects (font (size 1.27 1.27)) (justify right bottom))
+  )
+  (label "LS2" (at 105.41 64.77 0) (fields_autoplaced)
+    (effects (font (size 1.27 1.27)) (justify left bottom))
+  )
   (label "GND" (at 76.2 109.22 0) (fields_autoplaced)
     (effects (font (size 1.27 1.27)) (justify left bottom))
@@
     (effects (font (size 1.27 1.27)) (justify left bottom))
   )
+  (label "VDDIO" (at 104.14 91.44 0) (fields_autoplaced)
+    (effects (font (size 1.27 1.27)) (justify left bottom))
+  )
   (label "I2C_ADDR" (at 34.29 72.39 270) (fields_autoplaced)
     (effects (font (size 1.27 1.27)) (justify right bottom))
   )
+  (label "LS5" (at 106.68 72.39 0) (fields_autoplaced)
+    (effects (font (size 1.27 1.27)) (justify left bottom))
+  )
   (label "VDDIO" (at 55.88 97.79 0) (fields_autoplaced)
     (effects (font (size 1.27 1.27)) (justify left bottom))
   )
+  (label "LS1" (at 107.95 95.25 180) (fields_autoplaced)
+    (effects (font (size 1.27 1.27)) (justify right bottom))
+  )
+  (label "LS3" (at 107.95 100.33 180) (fields_autoplaced)
+    (effects (font (size 1.27 1.27)) (justify right bottom))
+  )
   (label "VDDIO" (at 156.21 26.67 0) (fields_autoplaced)
     (effects (font (size 1.27 1.27)) (justify left bottom))
@@
     (effects (font (size 1.27 1.27)) (justify right bottom))
   )
+  (label "LS3" (at 106.68 67.31 0) (fields_autoplaced)
+    (effects (font (size 1.27 1.27)) (justify left bottom))
+  )
   (label "SCL" (at 22.86 62.23 180) (fields_autoplaced)
     (effects (font (size 1.27 1.27)) (justify right bottom))
   )
+  (label "GND" (at 105.41 109.22 180) (fields_autoplaced)
+    (effects (font (size 1.27 1.27)) (justify right bottom))
+  )
   (label "SDA" (at 105.41 46.99 180) (fields_autoplaced)
     (effects (font (size 1.27 1.27)) (justify right bottom))
+  )
+  (label "LS4" (at 105.41 69.85 0) (fields_autoplaced)
+    (effects (font (size 1.27 1.27)) (justify left bottom))
   )
   (label "SDA" (at 24.13 53.34 90) (fields_autoplaced)
@@
         )
       )
+    )
+  )
+  (symbol (lib_id "Connector_Generic:Conn_01x07") (at 119.38 100.33 0) (unit 1)
+    (in_bom yes) (on_board yes) (dnp no) (fields_autoplaced)
+    (property "Reference" "J1" (at 121.92 99.695 0)
+      (effects (font (size 1.27 1.27)) (justify left))
+    )
+    (property "Value" "Conn_01x07" (at 121.92 102.235 0)
+      (effects (font (size 1.27 1.27)) (justify left))
+    )
+    (property "Footprint" "" (at 119.38 100.33 0)
+      (effects (font (size 1.27 1.27)) hide)
+    )
+    (property "Datasheet" "~" (at 119.38 100.33 0)
+      (effects (font (size 1.27 1.27)) hide)
+    )
+    (pin "1")
+    (pin "2")
+    (pin "3")
+    (pin "4")
+    (pin "5")
+    (pin "6")
+    (pin "7")
+    (instances
+      (project "Satellite_Circuit"
+        (path "/1ba48872-20f1-4135-8850-dcaa1bdd8874"
+          (reference "J1") (unit 1)
+        )
+      )
